File: hardware/phase1/stm32_board/stm32_official_prototype.kicad_sch (KiCad schematic)
At the start: 81 parts, among them CN11 Conn_02x36_Odd_Even, CN12 Conn_02x36_Odd_Even, CN14 USB_B_Micro, CN5 Conn_ARM_JTAG_SWD_10, U1 STM32L496ZGTx, U12 STMPS2151STR, U4 MMBT9013, U5 USBLC6-2SC6, U6 LD39050PU33R, U6 ST890CDR, U7 LD1117S50TR, U8 TSV631AILT, U9 ESDALC6V1W5

Commit message: Update stm32_official_prototype.kicad_sch
working on adding circuit breakers (0 ohm resistors) to each exposed pin
Parts:
- added SB124, SB130, SB131, SB132, SB142, SB143, SB171, SB197: Closed, RC0603N_YAG, symbol RC0603JR-070RL:RC0603JR-070RL
- added SB134, SB135, SB162, SB172: RC0603JR-070RL, RC0603N_YAG, symbol RC0603JR-070RL:RC0603JR-070RL
- renumbered U4 to T2, U6 to U4
Connections:
- net IOREF: now also B1.2, B1.3, R44.1
- net PA10: now also SB134.1, SB134.2
- net PA11: now also SB142.1, SB142.2
- net PA12: now also SB143.1, SB143.2
- net PA9: now also SB135.1; no longer R54.1
- net PB14: now also SB132.1; no longer R29.1
- net PB3: now also SB162.1
- net PB7: now also SB172.1; no longer R30.1
- net PC13: now also SB197.1; no longer R43.1
- net PC7: now also SB124.1; no longer R37.1
- net PG7: now also SB131.1
- net PG8: now also SB130.1
- net PH3-BOOT0: now also SB171.1; no longer R38.1
- new net: R37.1, SB124.2
- new net: R30.1, SB172.2
- new net: R29.1, SB132.2
- new net: R54.1, SB135.2
- new net: R43.1, SB197.2
- new net: R38.1, SB171.2
- new net STLK_RX: SB131.2
- new net STLK_TX: SB130.2
- new net SWO: SB162.2
Other:
- moved on the sheet: JP4, LD1, LD2, LD3, R29, R30, R31, R36, R37, R38, R54, U8

Commit message: Update stm32_official_prototype.kicad_sch
organized into sub-blocks
Parts:
- added C40: [N/A], symbol Device:C_Small
- added SB110, SB111, SB123, SB167: Open, RC0603N_YAG, symbol RC0603JR-070RL:RC0603JR-070RL
- added SB112, SB149, SB152, SB154, SB158: Closed, RC0603N_YAG, symbol RC0603JR-070RL:RC0603JR-070RL
- added SB198, SB199, SB200, SB201: RC0603JR-070RL, RC0603N_YAG, symbol RC0603JR-070RL:RC0603JR-070RL
- C45: value 100nF -> [N/A]
- L3: renamed from FB1; value FerriteBead_Small -> BEAD
Connections:
- net +3V3: now also SB110.1, SB111.1
- net AVDD: now also SB149.2, SB152.2; no longer C45.1, C56.1, C57.1, CN12.7 (Pin_7), L3.2, U1.32 (VREF+)
- net IOREF: now also SB110.2, SB111.2, SB112.2; no longer B1.2, B1.3, C28.1, C29.1, C30.1, C31.1, C32.1, C33.1, C34.1, C49.1, C50.1, C51.1, C52.1, C53.1, C54.1, C60.1, C61.1, CN11.33 (Pin_33), CN11.5 (Pin_5), CN5.1 (VTref), D2.1, JP5.2 (Pin_2), L3.1, R44.1, U1.106 (VDDUSB), U1.108 (VDD), U1.121 (VDD), U1.131 (VDDIO2), U1.144 (VDD), U1.17 (VDD), U1.39 (VDD), U1.52 (VDD), U1.6 (VBAT), U1.62 (VDD), U1.72 (VDD), U1.84 (VDD), U1.95 (VDDIO2)
- net PA5: now also SB123.1
- net PA9: no longer C42.1, CN14.1 (VBUS), R46.2, R49.1, R54.2, U12.1 (OUT), U5.5 (VBUS)
- net PG6: now also SB200.2, SB201.1; no longer R50.2
- net USB_OverCurrent: now also SB198.1; no longer LD7.1 (K), R51.2, U12.3 (FAULT)
- net VBUS_DET: now also SB199.1; no longer R46.1, R47.2
- net at R37.1, SB124.2: now also SB123.2
- net at B1.1, B1.4, R42.2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: now also C40.1; no longer R44.2
- net USB_PowerSwitchOn: no longer names the net of R52.2, U12.4 (EN)
- net USB_PowerSwitchOn: now also SB200.1
- new net: LD7.1 (K), R51.2, SB198.2, U12.3 (FAULT)
- new net: R50.2, SB201.2
- new net: L3.1, SB158.2, SB167.2
- new net: R46.1, R47.2, SB199.2
- new net: L3.2, SB152.1
- new net: C40.2, R44.2
- new net USB_VBUS: C42.1, CN14.1 (VBUS), R46.2, R49.1, R54.2, U12.1 (OUT), U5.5 (VBUS)
- new net VBAT: C60.1, CN11.33 (Pin_33), SB154.2, U1.6 (VBAT)
- new net VDD: C31.1, C50.1, C51.1, C52.1, CN11.5 (Pin_5), CN5.1 (VTref), D2.1, JP5.2 (Pin_2), SB158.1, U1.106 (VDDUSB), U1.131 (VDDIO2), U1.95 (VDDIO2)
- new net VDD_MCU: B1.2, B1.3, C28.1, C29.1, C30.1, C32.1, C33.1, C34.1, C49.1, C53.1, C54.1, C61.1, R44.1, SB112.1, SB154.1, SB167.1, U1.108 (VDD), U1.121 (VDD), U1.144 (VDD), U1.17 (VDD), U1.39 (VDD), U1.52 (VDD), U1.62 (VDD), U1.72 (VDD), U1.84 (VDD)
- new net VREF+: C45.1, C56.1, C57.1, CN12.7 (Pin_7), SB149.1, U1.32 (VREF+)
Other:
- note added: "POWER"
- note added: "STM32 uC"
- note added: "SWD"
- note added: "USB"
- moved on the sheet: B1, B2, C11, C16, C17, C18, C19, C20, C26, C27, C28, C29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

Commit message: Update stm32_official_prototype.kicad_sch
removed unnecessary circuitry
Parts:
- removed C11, C20, C26: 100nF, Capacitor,100nF,10%,16V,X7R,0603,YAGEO:CC0603N_YAG, symbol Device:C_Small
- removed C16, C42: 4.7uF, TAN Capacitor,4.7uF,10%,16V,A Type,AVX:TAJA_AVX, symbol Device:C_Polarized_Small
- removed C17: 10uF, TAN Capacitor,10uF,10%,16V,A Type,AVX:CAPMP3216X180N, symbol Device:C_Polarized_Small
- removed C18: 10uF(25V), Tan Capacitor,10uF,10%,25V,Tan-B,TAJB106K025RNJ:CAPMP3516X190N, symbol Device:C_Polarized_Small
- removed C19, C27: 1uF_X5R_0603, Capacitor,1uF,0603,16V,10%,X5R,YAGEO:CAPC1608X90, symbol Device:C_Small
- removed JP5: Conn_02x01, HDR_1x2_2R54:61300211121, symbol Connector_Generic:Conn_02x01
- removed JP6: Conn_02x04_Odd_Even, 2x4_2R54:61300821121, symbol Connector_Generic:Conn_02x04_Odd_Even
- removed LD5, LD7: Red, LED-SMD-RED-DIFFUSED_0603_:LED-0603, symbol Device:LED_Small
- removed LD6, LD8: Green, SMD-LED-CLEAR-GREEN_0603_:LED-0603, symbol Device:LED_Small
- removed R22, R28: 1K, RC0603FR-071KL:RESC1607X60N, symbol Device:R_Small
- removed R26, R52: 10K, RC0603FR-0710KL:RESC1607X60N, symbol Device:R_Small
- removed R27: 2K7, RES_2.7K_0603_:R0603, symbol Device:R_Small
- removed R41: 330, RC0603FR-07330RL:RESC1607X60N, symbol Device:R_Small
- removed R45: 620, RC0603FR-07620RL:RESC1608X55N, symbol Device:R_Small
- removed R48: 22K, RC0603FR-0722KL:RESC1607X60N, symbol Device:R_Small
- removed R49, R51: 47K, RC0603FR-0747KL:RESC1608X55, symbol Device:R_Small
- removed SB198, SB200: RC0603JR-070RL, RC0603N_YAG, symbol RC0603JR-070RL:RC0603JR-070RL
- removed T2: MMBT9013, MMBT9013:SOT-23, symbol MMBT9013:MMBT9013
- removed U12: STMPS2151STR, STMPS2151STR:SOT23-5L_STM, symbol 2025-01-04_16-51-05:STMPS2151STR
- removed U4: ST890CDR, ST890CDR:SO-8_STM, symbol 2025-01-04_17-43-57:ST890CDR
- removed U6: LD39050PU33R, LD39050PU33R:DFN6_3X3_STM, symbol 2025-01-04_20-45-34:LD39050PU33R
- removed U7: LD1117S50TR, LD1117S50TR:SOT230P700X180-4N, symbol LD1117S50TR:LD1117S50TR
- R46: footprint RC0603FR-07430KL:RESC1608X55N -> RC0603FR-071K5L:RESC1607X60N
- R47: footprint RC0603FR-07620KL:RESC1608X55N -> RC0603FR-071K5L:RESC1607X60N
- SB124, SB130, SB131, SB132, SB134, SB135, SB142, SB143, SB162, SB171, SB172, SB197: footprint RC0603N_YAG -> (none)
Connections:
- net VBUS_DET is gone; now on net PG5: SB199.1
- net +3V3: no longer SB110.1, U8.5 (VCC+)
- net PA12: now also R46.1
- net USB_VBUS: no longer R46.2
- net at R47.2, SB199.2: now also R46.2; no longer R46.1
- new net +3V3_PER: SB110.1, U8.5 (VCC+)
- no-connect marks 7 -> 5
Other:
- note added: "GPIO STATUS OUTPUT"
- note added: "GPIOs"
- note added: "POWER CTRL and RESET"
- moved on the sheet: CN14, D6, LD1, R31, R36, R37, R50, R54, SB123, SB124, SB134, SB135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

Commit message: stm32 board update (1.11.25)
- correcting footprints (IP)
- left off on USB circuitry
- note: net labels must be corrected for differential pair
Parts:
- removed C40: [N/A], symbol Device:C_Small
- removed C45: [N/A], HDR_1x2_2R54:61300211121, symbol Device:C_Small
- removed SB134: RC0603JR-070RL, symbol RC0603JR-070RL:RC0603JR-070RL
- added SB166: Closed, RC0603JR-070RL:RESC1607X60N, symbol RC0603JR-070RL:RC0603JR-070RL
- SB110, SB111, SB112, SB123, SB149, SB152, SB154, SB158, SB167, SB199, SB201: footprint RC0603N_YAG -> RC0603JR-070RL:RESC1607X60N
- SB124, SB130, SB131, SB132, SB135, SB142, SB143, SB162, SB172, SB197: footprint (none) -> RC0603JR-070RL:RESC1607X60N
- SB171: value Closed -> Circuit Breaker-SMPS; footprint (none) -> RC0603JR-070RL:RESC1607X60N
Connections:
- net GND: now also SB166.1, SB166.2
- net PA10: no longer CN14.4 (ID)
- net at B1.1, B1.4, R42.2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: now also R44.2
- no-connect marks 5 -> 6

Commit message: stm32 PCB board ~50% finished
- left off on verifying button footprint
(im trying to follow the original manufacturer BOM as much as possible, but some parts aren't downloadable.

- best solution is to use the notes column in the BOM, describes what the footprint is (SMT, 6x6mm, tactile switch, etc.)
Parts:
- B1, B2: footprint TS02-66-60-BK-160-LCR-D:SW_TS02-66-60-BK-160-LCR-D -> TS04_66_43_BK_260_SMT:SW_TS04-66-43-BK-260-SMT
Connections:
- net PH3-BOOT0: now also R38.1, SB171.2; no longer SB171.1, U1.138 (PH3)
- new net PH3: SB171.1, U1.138 (PH3)
Changed lines of the file:
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@@
 	)
 	(junction
+		(at 695.96 250.19)
+		(diameter 0)
+		(color 0 0 0 0)
+	)
+	(junction
 		(at 288.925 337.185)
 		(diameter 0)
@@
 	(wire
 		(pts
+			(xy 655.955 250.19) (xy 669.925 250.19)
+		)
+		(stroke
+			(width 0)
+			(type default)
+		)
+	)
+	(wire
+		(pts
 			(xy 580.39 41.91) (xy 590.55 41.91)
 		)
@@
 	(wire
 		(pts
-			(xy 669.925 250.19) (xy 666.115 250.19)
-		)
-		(stroke
-			(width 0)
-			(type default)
-		)
-	)
-	(wire
-		(pts
 			(xy 717.55 71.755) (xy 714.375 71.755)
 		)
@@
 	(wire
 		(pts
+			(xy 695.96 250.19) (xy 709.295 250.19)
+		)
+		(stroke
+			(width 0)
+			(type default)
+		)
+	)
+	(wire
+		(pts
 			(xy 690.88 44.45) (xy 680.085 44.45)
 		)
@@
 		)
 	)
+	(global_label "PH3"
+		(shape bidirectional)
+		(at 655.955 250.19 180)
+		(fields_autoplaced yes)
+		(effects
+			(font
+				(size 1.27 1.27)
+			)
+			(justify right)
+		)
+		(property "Intersheetrefs" "${INTERSHEET_REFS}"
+			(at 648.0485 250.19 0)
+			(effects
+				(font
+					(size 1.27 1.27)
+				)
+				(justify right)
+				(hide yes)
+			)
+		)
+	)
 	(global_label "PG4"
 		(shape bidirectional)
@@
 		)
 	)
-	(global_label "PH3-BOOT0"
+	(global_label "PH3"
 		(shape bidirectional)
 		(at 51.435 80.01 180)
@@
 		)
 		(property "Intersheetrefs" "${INTERSHEET_REFS}"
-			(at 35.848 80.01 0)
+			(at 43.5285 80.01 0)
 			(effects
 				(font
@@
 	(global_label "PH3-BOOT0"
 		(shape bidirectional)
-		(at 666.115 250.19 180)
+		(at 709.295 250.19 0)
 		(fields_autoplaced yes)
 		(effects
@@
 				(size 1.27 1.27)
 			)
-			(justify right)
+			(justify left)
 		)
 		(property "Intersheetrefs" "${INTERSHEET_REFS}"
-			(at 650.528 250.19 0)
+			(at 724.882 250.19 0)
 			(effects
 				(font
 					(size 1.27 1.27)
 				)
-				(justify right)
+				(justify left)
 				(hide yes)
 			)
@@
 			)
 		)
-		(property "Footprint" "TS02-66-60-BK-160-LCR-D:SW_TS02-66-60-BK-160-LCR-D"
+		(property "Footprint" "TS04_66_43_BK_260_SMT:SW_TS04-66-43-BK-260-SMT"
 			(at 99.06 311.785 90)
 			(effects
@@
 			)
 		)
-		(property "Footprint" "TS02-66-60-BK-160-LCR-D:SW_TS02-66-60-BK-160-LCR-D"
+		(property "Footprint" "TS04_66_43_BK_260_SMT:SW_TS04-66-43-BK-260-SMT"
 			(at 99.06 363.22 90)
 			(effects

Commit message: stm32 pcb update for (1.13.25)
- most components are now connected
- need to verify a few more footprints
- board is ~65% finished
Parts:
- renumbered CN5 to SWD, U5 to U13
Connections:
- net PA12: no longer R46.1
- net USB_VBUS: now also R46.1
Changed lines of the file:
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@@
 	)
 	(junction
-		(at 717.55 58.42)
+		(at 582.93 83.185)
 		(diameter 0)
 		(color 0 0 0 0)
 	)
 	(junction
-		(at 582.93 83.185)
+		(at 721.995 64.135)
 		(diameter 0)
 		(color 0 0 0 0)
@@
 	(wire
 		(pts
-			(xy 713.74 44.45) (xy 717.55 44.45)
+			(xy 713.74 44.45) (xy 721.995 44.45)
 		)
 		(stroke
@@
 		)
 	)
-	(wire
-		(pts
-			(xy 717.55 44.45) (xy 717.55 58.42)
-		)
-		(stroke
-			(width 0)
-			(type default)
-		)
-	)
 	(polyline
 		(pts
@@
 	(wire
 		(pts
+			(xy 721.995 44.45) (xy 721.995 64.135)
+		)
+		(stroke
+			(width 0)
+			(type default)
+		)
+	)
+	(wire
+		(pts
 			(xy 588.645 83.185) (xy 582.93 83.185)
 		)
@@
 		)
 	)
+	(label "GND"
+		(at 307.975 120.015 0)
+		(fields_autoplaced yes)
+		(effects
+			(font
+				(size 1.27 1.27)
+			)
+			(justify left bottom)
+		)
+	)
 	(label "Diff Pair (-) 90ohm"
 		(at 491.49 61.595 0)
@@
 		(dnp no)
 		(fields_autoplaced yes)
-		(property "Reference" "U5"
+		(property "Reference" "U13"
 			(at 723.6461 73.66 0)
 			(effects
@@
 			(project ""
 				(path "/eb5365fc-f6b5-4558-a59a-9210174c0865"
-					(reference "U5")
+					(reference "U13")
 					(unit 1)
 				)
@@
 		(dnp no)
 		(fields_autoplaced yes)
-		(property "Reference" "CN5"
+		(property "Reference" "SWD"
 			(at 514.35 219.7099 0)
 			(effects
@@
 			(project ""
 				(path "/eb5365fc-f6b5-4558-a59a-9210174c0865"
-					(reference "CN5")
+					(reference "SWD")
 					(unit 1)
 				)

Commit message: STM32 board update (1.25.25)
- vastly improved the layout
- verified ALL footprints
- implemented correct JLCPCB design rules
- left off on labeling
Parts:
- removed D2: SMLVT3V3, SMLVT3V3:SMB_STM, symbol 2025-01-08_22-06-10:SMLVT3V3
- removed D6: ESDALC6V1-1U2, ESDALC6V1-1U2:DIODE_ESDALC6V1-1U2, symbol ESDALC6V1-1U2:ESDALC6V1-1U2
- removed JP4: Conn_02x01, HDR_1x2_2R54:61300211121, symbol Connector_Generic:Conn_02x01
- removed R54: 10K, RC0603FR-0710KL:RESC1607X60N, symbol Device:R_Small
- removed SB135, SB162: RC0603JR-070RL, RC0603JR-070RL:RESC1607X60N, symbol RC0603JR-070RL:RC0603JR-070RL
- removed SB171: Circuit Breaker-SMPS, RC0603JR-070RL:RESC1607X60N, symbol RC0603JR-070RL:RC0603JR-070RL
- added C40, C45: [N/A], CC0603KRX7R7BB104:CAPC1608X90, symbol Device:C_Small
- added D2: SMLVT3V3, SMLVT3V3:DIOM4336X265N, symbol Device:D_Small
- added D6: ESDALC6V1-1U2, ESDALC6V1-1U2:DIODE_ESDALC6V1-1U2, symbol Device:D_Small
- added JP4: Conn_01x02_Pin, Connector_PinHeader_2.54mm:PinHeader_1x02_P2.54mm_Vertical, symbol Connector:Conn_01x02_Pin
- added LD8: Green, SMD-LED-CLEAR-GREEN_0603_:LED-0603, symbol Device:LED_Small
- added R41: 330, RC0603FR-07330RL:RESC1607X60N, symbol Device:R_Small
- added R48: 22K, RC0603FR-0722KL:RESC1607X60N, symbol Device:R_Small
- added R49: 47K, RC0603FR-0747KL:RESC1608X55, symbol Device:R_Small
- added SB119: Open, RC0603JR-070RL:RESC1607X60N, symbol RC0603JR-070RL:RC0603JR-070RL
- added T2: 9013, MMBT9013:SOT-23, symbol MMBT9013:MMBT9013
- C28, C29, C30, C31, C32, C33, C34, C41, C49, C50, C51, C53, C57, C58, C61: footprint Capacitor,100nF,10%,16V,X7R,0603,YAGEO:CC0603N_YAG -> CC0603KRX7R7BB104:CAPC1608X90
- C52, C54: footprint Capacitor，4.7uF，16V， X5R，10%，0603:CAPC1608X90 -> CC0603KRX5R7BB475:CAPC1608X90
- C56, C59: footprint TAN Capacitor,1uF,10%,16V,A Type,AVX:CAPMP3216X180N -> TAJA105K016R:CAPMP3216X166
- C60: footprint Capacitor,1uF,0603,16V,10%,X5R,YAGEO:CAPC1608X90 -> CC0603KRX5R7BB105:CAPC1608X90
- CN11, CN12: footprint SLM-136-01-S-D:SAMTEC_SLM-136-01-S-D -> Connector_PinSocket_2.54mm:PinSocket_2x36_P2.54mm_Vertical
- CN5: renamed from SWD; footprint SSW_105_06_G_D:SAMTEC_SSW-105-06-G-D -> Connector_PinSocket_2.54mm:PinSocket_2x05_P2.54mm_Vertical
- L3: footprint FERRITEBEAD_0603:CAPC1608X90N -> FCM1608KF-601T05:FB0603
- R30: footprint RES-680R-0603_:R0603 -> SMD-RES-680R-1_-1_10W_0603_:R0603
- R46: footprint RC0603FR-071K5L:RESC1607X60N -> RC0603FR-07430KL:RESC1608X55N
- R47: footprint RC0603FR-071K5L:RESC1607X60N -> RC0603FR-07620KL:RESC1608X55N
- SB172, SB199, SB201: value RC0603JR-070RL -> Closed
- U11: renamed from U1; footprint Package_QFP:LQFP-144_20x20mm_P0.5mm -> STM32L496ZGT6:LQFP144-20x20mm_STM
- U13: footprint Package_TO_SOT_SMD:SOT-23-6 -> USBLC6-2SC6:SOT95P280X145-6N
- U9: footprint ESDALC6V1W5:SOT323-5L -> ESDALC6V1W5:SOT65P210X110-5N
Connections:
- net PH3 is gone; now on net PH3-BOOT0: U11.138 (PH3)
- net USB_VBUS is gone; now on net PA9: CN14.1 (VBUS), R46.1, U13.5 (VBUS)
- net +3V3_PER: now also R41.2
- net GND: now also D2.2 (A), D6.2 (A), R48.2, T2.2; no longer C56.2, C57.2, C58.2, C59.2, CN12.32 (Pin_32), SB166.2, U11.30 (VSSA), U11.31 (VREF-)
- net PA10: now also CN14.4 (ID), D6.1 (K)
- net PA11: no longer CN14.2 (D-), SB142.2, U13.1 (I/O1), U13.6 (I/O1)
- net PA12: no longer CN14.3 (D+), R50.1, SB143.2, U13.3 (I/O2), U13.4 (I/O2)
- net PA9: now also R49.1
- net VDD: now also D2.1 (K)
- net VREF+: now also C45.1, SB119.2; no longer CN12.7 (Pin_7)
- net at B1.1, B1.4, R42.2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: now also C40.1; no longer R44.2
- net PG5 renamed PG5 (VBUS_DET)
- net PG5 (VBUS_DET): now also JP4.1 (Pin_1); no longer SB199.1
- net PG6 renamed PG6 (USB_Disconnect)
- new net: C40.2, R44.2
- new net: LD8.2 (A), R41.1
- new net: R48.1, R49.2, T2.1
- new net: CN12.7 (Pin_7), SB119.1
- new net: LD8.1 (K), T2.3
- new net GNDA: C45.2, C56.2, C57.2, C58.2, C59.2, CN12.32 (Pin_32), SB166.2, U11.30 (VSSA), U11.31 (VREF-)
- new net USB_DM: CN14.2 (D-), SB142.2, U13.1 (I/O1), U13.6 (I/O1)
- new net USB_DP: CN14.3 (D+), R50.1, SB143.2, U13.3 (I/O2), U13.4 (I/O2)
- new net VBUS_DET: JP4.2 (Pin_2), SB199.1
- no-connect marks 6 -> 5

Commit message: toreyin meeting stm32 board update (1.29.25)
- I MUST NOT FORGET DIFFERENTIAL ROUTING FOR USB
- i need like 10 pins to wire, difficult at this point to get through the entire spider web of traces
- buttons, USB, LEDs, and power network need to be connected to main circuit
- we for sure ordering this week
Parts:
- removed SB130, SB131: Closed, RC0603JR-070RL:RESC1607X60N, symbol RC0603JR-070RL:RC0603JR-070RL
Connections:
- net PB7: now also R30.1, SB172.2; no longer SB172.1, U11.137 (PB7)
- new net: SB172.1, U11.137 (PB7)
Other:
- moved on the sheet: SB172, SB197
