File: hardware/phase1/stm32_board/stm32_official_prototype.kicad_sch (KiCad schematic)
At the start: 75 parts, among them CN11 Conn_02x36_Odd_Even, CN12 Conn_02x36_Odd_Even, CN14 USB_B_Micro, CN5 Conn_ARM_JTAG_SWD_10, T2 9013, U11 STM32L496ZGTx, U13 USBLC6-2SC6, U8 TSV631AILT, U9 ESDALC6V1W5

Commit message: legit stm32 schematic (2.8.25)
- removed most if not all redundant short breakers
- implemented extra safeguard for temporary power supply
- BOARD IS SUPPLIED THROUGH +3V3  pin 16 on connector CN11
Parts:
- removed C45: [N/A], CC0603KRX7R7BB104:CAPC1608X90, symbol Device:C_Small
- removed JP4: Conn_01x02_Pin, Connector_PinHeader_2.54mm:PinHeader_1x02_P2.54mm_Vertical, symbol Connector:Conn_01x02_Pin
- removed R46: 430K, RC0603FR-07430KL:RESC1608X55N, symbol Device:R_Small
- removed R47: 620K, RC0603FR-07620KL:RESC1608X55N, symbol Device:R_Small
- removed R50: 1K5, RC0603FR-071K5L:RESC1607X60N, symbol Device:R_Small
- removed SB110, SB119, SB123, SB167: Open, RC0603JR-070RL:RESC1607X60N, symbol RC0603JR-070RL:RC0603JR-070RL
- removed SB199, SB201: Closed, RC0603JR-070RL:RESC1607X60N, symbol RC0603JR-070RL:RC0603JR-070RL
- added C19, C27: 1uF, CC0603KRX5R7BB105:CAPC1608X90, symbol Device:C_Small
- added C20, C26: 100nF, CC0603KRX7R7BB104:CAPC1608X90, symbol Device:C_Small
- added C42: 4.7uF, TAJA475K016R:CAPMP3216X166, symbol Device:C_Polarized_Small
- added JP5: Conn_01x02_Pin, Connector_PinHeader_2.54mm:PinHeader_1x02_P2.54mm_Vertical, symbol Connector:Conn_01x02_Pin
- added LD6: Green, SMD-LED-CLEAR-GREEN_0603_:LED-0603, symbol Device:LED_Small
- added LD7: Red, LED-SMD-RED-DIFFUSED_0603_:LED-0603, symbol Device:LED_Small
- added R28: 1K, RC0603FR-071KL:RESC1607X60N, symbol Device:R_Small
- added R45: 620, RC0603FR-07620RL:RC0603N_YAG, symbol Device:R_Small
- added R51: 47K, RC0603FR-0747KL:RESC1608X55, symbol Device:R_Small
- added R52: 10K, RC0603FR-0710KL:RESC1607X60N, symbol Device:R_Small
- added SB6: Closed, RC0603JR-070RL:RESC1607X60N, symbol RC0603JR-070RL:RC0603JR-070RL
- added U1: STMPS2151STR, STMPS2151STR:SOT95P280X145-5N, symbol STMPS2151STR:STMPS2151STR
- added U2: LD39050PU33R, LD39050PU33R:SON95P300X300X100-7N, symbol LD39050PU33R:LD39050PU33R
- SB111: value Open -> Closed
Connections:
- net +3V3: now also R41.2, C27.1, R28.1, R45.2, R51.2, U2.6 (VIN); no longer SB111.1
- net GND: now also C19.2, C20.2, C26.2, C27.2, C42.2, LD6.1 (K), R52.1, U1.2 (GND), U2.2 (GND), U2.7 (GND)
- net PA9: now also C42.1, U1.1 (OUT)
- net VDD: now also SB111.1, U8.5 (VCC+), JP5.2 (Pin_2), U1.5 (IN)
- net VREF+: now also CN12.7 (Pin_7)
- removed net +3V3_PER: R41.2, U8.5 (VCC+)
- net PG5 (VBUS_DET) renamed PG5
- net PG6 (USB_Disconnect) renamed PG6
- new net: LD6.2 (A), R28.2
- new net: JP5.1 (Pin_1), SB6.2
- new net: LD7.1 (K), R51.1, U1.3 (~{FAULT})
- new net: R52.2, U1.4 (EN)
- new net: C26.1, U2.1 (EN)
- new net: LD7.2 (A), R45.1
- new net: C19.1, C20.1, SB6.1, U2.4 (VOUT)
- no-connect marks 5 -> 6
Other:
- moved on the sheet: CN14, D6, L3, LD8, R41, R48, R49, SB158, T2, U13

Commit message: layout finish, clearing all DRC errors stm32 update (2.9.25)
Parts:
- removed SB111, SB112, SB149, SB152, SB154, SB158, SB166: Closed, RC0603JR-070RL:RESC1607X60N, symbol RC0603JR-070RL:RC0603JR-070RL
- added R54: 10K, RC0603FR-0710KL:RESC1607X60N, symbol Device:R_Small
- added SB135: Closed, RC0603JR-070RL:RESC1607X60N, symbol RC0603JR-070RL:RC0603JR-070RL
- renumbered U1 to U12, U2 to U6
Connections:
- net GNDA is gone; now on net GND: C56.2, C57.2, C58.2, C59.2, CN12.32 (Pin_32), U11.30 (VSSA), U11.31 (VREF-)
- net VBAT is gone; now on net VDD: C60.1, CN11.33 (Pin_33), U11.6 (VBAT)
- net VDD_MCU is gone; now on net VDD: B1.2, B1.3, C28.1, C29.1, C30.1, C32.1, C33.1, C34.1, C49.1, C53.1, C54.1, C61.1, R44.1, U11.108 (VDD), U11.121 (VDD), U11.144 (VDD), U11.17 (VDD), U11.39 (VDD), U11.52 (VDD), U11.62 (VDD), U11.72 (VDD), U11.84 (VDD)
- net VREF+ is gone; now on net AVDD: C56.1, C57.1, CN12.7 (Pin_7), U11.32 (VREF+)
- net +3V3: no longer R41.2, R45.2, R51.2
- net AVDD: now also L3.2
- net PA9: now also SB135.1; no longer C42.1, CN14.1 (VBUS), R49.1, U12.1 (OUT), U13.5 (VBUS)
- net VDD: now also L3.1, R41.2, R45.2, R51.2
- net USB_DM renamed USB_DN
- new net: R54.1, SB135.2
- new net USB_VBUS: C42.1, CN14.1 (VBUS), R49.1, R54.2, U12.1 (OUT), U13.5 (VBUS)
