File: LTC3556_v1.2a.kicad_sch (KiCad schematic)
At the start: 43 parts, among them J1 USB_B_Micro, J2 Conn_01x01_Pin, J3 Conn_01x01_Pin, J4 Conn_01x01_Pin, J5 Conn_01x01_Pin, J6 Conn_01x01_Pin, Q1 SI2333DS-T1-E3, SW1 SW_SPDT, U1 LTC3556EUFD_PBF

Commit message: Add files via upload
-Added TC7660EOA charge pump for AFE -2.5V AVSS
- Ppdated integration of both U1 and U2 IC's, V_Out I/O connections.
Parts:
- added C15, C16, C17: 10uF, Capacitor_SMD:C_0805_2012Metric_Pad1.18x1.45mm_HandSolder, symbol Device:C
- added D1: LED, LED_SMD:LED_0805_2012Metric_Pad1.15x1.40mm_HandSolder, symbol Device:LED
- added J10, J11, J13, J15, J7, J8, J9: Conn_01x01_Pin, Connector_PinSocket_1.27mm:PinSocket_1x01_P1.27mm_Vertical, symbol Connector:Conn_01x01_Pin
- added J12: Conn_01x02_Pin, Connector_JST:JST_EH_S2B-EH_1x02_P2.50mm_Horizontal, symbol Connector:Conn_01x02_Pin
- added J14: Conn_01x01_Pin, Connector_PinHeader_1.27mm:PinHeader_1x01_P1.27mm_Vertical, symbol Connector:Conn_01x01_Pin
- added R5: 510, Resistor_SMD:R_0402_1005Metric_Pad0.72x0.64mm_HandSolder, symbol Device:R_US
- added U2: ~, Package_SO:SO-8_3.9x4.9mm_P1.27mm, symbol TC7660EOA_LT3556_v1.2a_sym:TC7660EOA
- J2, J3, J4, J5, J6: footprint Connector_PinHeader_1.27mm:PinHeader_1x01_P1.27mm_Vertical -> Connector_PinSocket_1.27mm:PinSocket_1x01_P1.27mm_Vertical
- R10: value 365K -> 235K
- R9: value 365K -> 347K
Connections:
- net GND: now also H1.1, H2.1, H3.1, H4.1, C16.1, C17.2, D1.1 (K), J10.1 (Pin_1), J11.1 (Pin_1), J12.2 (Pin_2), J14.1 (Pin_1), U2.3 (GND), U2.6 (LV)
- net VBAT: now also J12.1 (Pin_1)
- net VOUT0: now also J13.1 (Pin_1)
- net VOUT1: now also J9.1 (Pin_1)
- net VOUT2: now also J8.1 (Pin_1)
- net at C13.1, L7.1, Q1.2 (S)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: now also R5.1
- net VOUT3: now reaches C11.1, C6.2, C7.2, R8.1, U1.12 (VOUT3), U1.18 (VIN2), U1.5 (VIN1)
- net VOUT3: now also J7.1 (Pin_1)
- net at C4.2, J6.1 (Pin_1), U1.1 (LDO3V3)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: now also C17.1, U2.8 (V+)
- new net: C15.1, U2.2 (CAP+)
- new net: C15.2, U2.4 (CAP-)
- new net: C16.2, J15.1 (Pin_1), U2.5 (V_OUT2.5V)
- new net: D1.2 (A), R5.2
- no-connect marks 4 -> 5
Other:
- note added: "+2.5V VOUT1"
- note added: "+3.3V"
- note added: "3.56V"
- note added: "5V input power"
- note added: "All logic input all 3 switching reg"
- note added: "Charge controll thur"
- note added: "ENALL"
- note added: "GND"
- note added: "High output sig"
- note added: "If USB disconn, battery power sys"
- note added: "If USB is connected the sys priorit USB power , chrge battery"
- note added: "Input"
- note added: "Logic Output open drain"
- note added: "MLCC (low ESR)"
- note added: "Match DV_cc to STM32 logic"
- note added: "Power Trans Pin Buck Switching Reg 1"
- note added: "Power Trans Pin Buck Switching Reg 2"
- note added: "Switching PowerPath as needed"
- note added: "USB auto switch between USB and battery"
- note added: "VBAT"
- note added: "VBAT (+)battery input supply power when USB unplugged"
- note added: "VOUT (-2.5V) to AVSS"
- note added: "VOUT2"
- note added: "VOUT3 Reg Buck Boost"
- note added: "always -On"
- note added: "battery charge status"
- moved on the sheet: C1, C10, C11, C12, C13, C14, C2, C3, C4, C5, C6, C7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
