File: hardware/phase1/pmic_board/LTC3556_v2.3.kicad_sch (KiCad schematic)
At the start: 67 parts, among them J1 USB_B_Micro, J10 Conn_01x01_Pin, J11 Conn_01x01_Pin, J12 Conn_01x02_Pin, J13 Conn_01x03_Pin, J14 Conn_01x01_Pin, J15 Conn_01x01_Pin, J16 Conn_01x01_Pin, J17 Conn_01x01_Pin, J18 Screw_Terminal_01x02, J19 Conn_01x02_Pin, J2 Conn_01x01_Pin, J20 Screw_Terminal_01x04, J21 Screw_Terminal_01x02, J3 Conn_01x01_Pin, J4 Conn_01x01_Pin, J5 Conn_01x01_Pin, J6 Conn_01x01_Pin, J7 Conn_01x01_Pin, J8 Conn_01x01_Pin, J9 Conn_01x01_Pin, Q1 SI2333DS, SW1 SW_SPDT, U1 LTC3556EUFD_PBF, U2 TC7660B

Commit message: Update LTC to add JLC MPNs and fix JST plug
Parts:
- J1: MPN (none) -> C10418
- J12: footprint Connector_JST:JST_EH_S2B-EH_1x02_P2.50mm_Horizontal -> Connector_JST:JST_PH_S2B-PH-K_1x02_P2.00mm_Horizontal; MPN (none) -> C173752
- J20: MPN (none) -> C474922
- J21: MPN (none) -> C474920
- SW1: MPN (none) -> C480342
- U1: MPN (none) -> C685032
- U2: MPN (none) -> C512761
Changed lines of the file:
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@@
 			)
 		)
+		(property "MPN" "C480342"
+			(at 351.79 60.96 0)
+			(effects
+				(font
+					(size 1.27 1.27)
+				)
+				(hide yes)
+			)
+		)
 		(pin "3"
 		)
@@
 			)
 		)
+		(property "MPN" "C10418"
+			(at 125.73 74.93 0)
+			(effects
+				(font
+					(size 1.27 1.27)
+				)
+				(hide yes)
+			)
+		)
 		(pin "2"
 		)
@@
 			)
 		)
+		(property "MPN" "C474922"
+			(at 396.24 116.84 0)
+			(effects
+				(font
+					(size 1.27 1.27)
+				)
+				(hide yes)
+			)
+		)
 		(pin "1"
 		)
@@
 			)
 		)
+		(property "MPN" "C685032"
+			(at 213.36 63.5 0)
+			(effects
+				(font
+					(size 1.27 1.27)
+				)
+				(hide yes)
+			)
+		)
 		(pin "3"
 		)
@@
 			)
 		)
+		(property "MPN" "C512761"
+			(at 60.96 77.47 0)
+			(effects
+				(font
+					(size 1.27 1.27)
+				)
+				(hide yes)
+			)
+		)
 		(pin "1"
 		)
@@
 			)
 		)
-		(property "Sim.Type" ""
+		(property "Sim.Type" "C474920"
 			(at 396.24 133.35 0)
 			(effects
@@
 			)
 		)
-		(property "Footprint" "Connector_JST:JST_EH_S2B-EH_1x02_P2.50mm_Horizontal"
+		(property "Footprint" "Connector_JST:JST_PH_S2B-PH-K_1x02_P2.00mm_Horizontal"
 			(at 396.24 83.82 0)
 			(effects
@@
 			)
 		)
+		(property "MPN" "C173752"
+			(at 396.24 83.82 0)
+			(effects
+				(font
+					(size 1.27 1.27)
+				)
+				(hide yes)
+			)
+		)
 		(pin "1"
 		)
@@
 			(at 396.24 60.96 0)
 			(effects
+				(font
+					(size 1.27 1.27)
+				)
+				(hide yes)
+			)
+		)
+		(property "MPN" "C474920"
+			(at 396.24 60.96 0)
+			(effects

Commit message: Update PMIC board: edit resistor values, added MPN numbers, fixed headers
Parts:
- removed J10, J11, J15, J16, J17, J2, J3, J4, J5, J6, J7, J8, J9: Conn_01x01_Pin, Connector_PinSocket_2.54mm:PinSocket_1x01_P2.54mm_Vertical, symbol Connector:Conn_01x01_Pin
- added J22: Conn_01x07, Connector_PinSocket_2.54mm:PinSocket_1x07_P2.54mm_Vertical, symbol Connector_Generic:Conn_01x07
- added J23: Conn_01x04, Connector_PinSocket_2.54mm:PinSocket_1x04_P2.54mm_Vertical, symbol Connector_Generic:Conn_01x04
- added J24: Conn_01x02, Connector_PinSocket_2.54mm:PinSocket_1x02_P2.54mm_Vertical, symbol Connector_Generic:Conn_01x02
- C17: value DNI -> DNP
- J13: MPN (none) -> C49257
- J14: MPN (none) -> C492400
- J18: MPN (none) -> C474920
- J19: MPN (none) -> C225477
- R10: value 235K -> 240K
- R11, R12, R13: value 111K -> 110K
- R9: value 347K -> 350K
- TH1: value 100K -> DNP
Connections:
- net GND: now also J23.4 (Pin_4), J24.2 (Pin_2)
- net SCL: now reaches U1.13 (SCL)
- net SCL: now also J22.6 (Pin_6)
- net CHRG: now reaches D2.1 (K), U1.21 (*CHRG)
- net CHRG: now also J22.3 (Pin_3)
- net 3V56: now reaches C11.1, C6.2, C7.2, R8.1, U1.12 (VOUT3), U1.18 (VIN2), U1.5 (VIN1)
- net 3V56: now also J22.1 (Pin_1)
- net 3V3: now reaches C12.1, C9.1, J18.1 (Pin_1), J20.3 (Pin_3), L2.1, R9.1
- net 3V3: now also J23.3 (Pin_3), J24.1 (Pin_1)
- net N2V5: now reaches J20.1 (Pin_1), U2.5 (VOUT)
- net N2V5: now also J23.1 (Pin_1)
- net P2V5: now reaches C10.1, C14.1, J20.2 (Pin_2), L3.1, R10.1
- net P2V5: now also J23.2 (Pin_2)
- net PGOOD: now reaches R3.2, U1.15 (PGOODALL)
- net PGOOD: now also J22.2 (Pin_2)
- net DVCC: now reaches C4.2, J13.1 (Pin_1), U1.10 (DVCC)
- net DVCC: now also J22.7 (Pin_7)
- net SDA: now reaches U1.16 (SDA)
- net SDA: now also J22.5 (Pin_5)
- net ENALL: now reaches U1.28 (ENALL)
- net ENALL: now also J22.4 (Pin_4)
Other:
- note added: "235K -> 240K"
- note added: "347K -> 350K"
- note added: "R11,12,13 (111K -> 110K)"
- moved on the sheet: C11, C12, C14, R11, R12, R13
