File: hardware/phase1/pmic_board/LTC3556_v2.4.kicad_sch (KiCad schematic)
At the start: 57 parts, among them J1 USB_B_Micro, J12 Conn_01x02_Pin, J13 Conn_01x03_Pin, J14 Conn_01x01_Pin, J18 Screw_Terminal_01x02, J19 Conn_01x02_Pin, J20 Screw_Terminal_01x04, J21 Screw_Terminal_01x02, J22 Conn_01x07, J23 Conn_01x04, J24 Conn_01x02, Q1 SI2333DS, SW1 SW_SPDT, U1 LTC3556EUFD_PBF, U2 TC7660B

Commit message: Fix PMIC files
Parts:
- R9: footprint Resistor_SMD:R_0402_1005Metric_Pad0.72x0.64mm_HandSolder -> Resistor_SMD:R_0603_1608Metric
Connections:
- net VOUT0: now reaches C18.1, C5.2, J21.1 (Pin_1), R1.1, R3.1, SW1.2 (B), U1.11 (VIN3), U2.8 (V+)
Other:
- note added: "+2.5V (VOUT1)"
- note added: "+3.56 (VOUT3)"
- note added: "AVSS Power"
- note added: "BATTERY"
- note added: "Pin Sockets"
- note added: "STM32_PWR"
- note added: "Terminal Blocks"
- note removed: "+2.5V VOUT1"
- note removed: "235K -> 240K"
- note removed: "3.56V"
- note removed: "347K -> 350K"
- note removed: "R11,12,13 (111K -> 110K)"
- note removed: "STM32_PWR +3v3 (VOUT2) GND"
- note removed: "VBAT (+)battery input supply power when USB unplugged"
- note removed: "VOUT3"
- moved on the sheet: C1, C10, C11, C12, C13, C14, C15, C16, C17, C18, C2, C3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
