File: hardware/phase1/ads1299_board/ads1299_official_prototype/ads1299_official_prototype.kicad_pcb (KiCad board)
At the start: 4 copper layers, 96 x 91 mm, 113 parts, among them IC1 ADS1299-4PAGR, J2 1725656, J3 TSM-110-01-T-DV-P-TR, J5 TSW-103-07-T-D, J6 36PIN_IDC, J9 1725656, U10 24AA256-I/ST, U11 OPA376AID, U4 OPA376

Commit message: Only official prototype file, fully finalized with BOM
Parts:
- R23, R24: value 0 -> 2.0M
Changed lines of the file:
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@@
 			)
 		)
-		(property "Value" "0"
+		(property "Value" "2.0M"
 			(at 1.908858 1.272555 0)
 			(layer "F.Fab")
@@
 			)
 		)
-		(property "Value" "0"
+		(property "Value" "2.0M"
 			(at 1.908858 1.272555 90)
 			(layer "F.Fab")
