File: hardware/phase1/ads1299_board/ads1299_official_prototype/ads1299_official_prototype.kicad_sch (KiCad schematic)
At the start: 108 parts, among them IC1 ADS1299-4PAGR, J2 1725656, J3 TSM-110-01-T-DV-P-TR, J5 TSW-103-07-T-D, J6 36PIN_IDC, J9 1725656, U10 24AA256-I/ST, U11 OPA376AID, U4 OPA376

Commit message: Only official prototype file, fully finalized with BOM
Parts:
- added Y1: FNGEPO002, FNGEPO002, symbol FNGEPO002:FNGEPO002
- R23, R24: value 0 -> 2.0M
Changed lines of the file:
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@@
 			)
 		)
-		(property "Value" "0"
+		(property "Value" "2.0M"
 			(at 213.36 274.3199 90)
 			(effects
@@
 			)
 		)
-		(property "Value" "0"
+		(property "Value" "2.0M"
 			(at 213.36 292.0999 90)
 			(effects
@@
 					(unit 1)
 				)
+			)
+		)
+	)
+	(symbol
+		(lib_id "FNGEPO002:FNGEPO002")
+		(at 347.98 346.71 0)
+		(unit 1)
+		(exclude_from_sim no)
+		(in_bom yes)
+		(on_board yes)
+		(dnp no)
+		(fields_autoplaced yes)
+		(property "Reference" "Y1"
+			(at 372.11 339.09 0)
+			(effects
+				(font
+					(size 1.27 1.27)
+				)
+			)
+		)
+		(property "Value" "FNGEPO002"
+			(at 372.11 341.63 0)
+			(effects
+				(font
+					(size 1.27 1.27)
+				)
+			)
+		)
+		(property "Footprint" "FNGEPO002"
+			(at 392.43 441.63 0)
+			(effects
+				(font
+					(size 1.27 1.27)
+				)
+				(justify left top)
+				(hide yes)
+			)
+		)
+		(property "Datasheet" "https://media.digikey.com/pdf/Data%20Sheets/Diodes%20PDFs/FNGEPO002.pdf"
+			(at 392.43 541.63 0)
+			(effects
+				(font
+					(size 1.27 1.27)
+				)
+				(justify left top)
+				(hide yes)
+			)
+		)
+		(property "Description" "Standard Clock Oscillators 2.048 MHz, 3.3V CMOS G/EPON VoIP"
+			(at 347.98 346.71 0)
+			(effects
+				(font
+					(size 1.27 1.27)
+				)
+				(hide yes)
+			)
+		)
+		(property "Height" "1.55"
+			(at 392.43 741.63 0)
+			(effects
+				(font
+					(size 1.27 1.27)
+				)
+				(justify left top)
+				(hide yes)
+			)
+		)
+		(property "Manufacturer_Name" "Diodes Incorporated"
+			(at 392.43 841.63 0)
+			(effects
+				(font
+					(size 1.27 1.27)
+				)
+				(justify left top)
+				(hide yes)
+			)
+		)
+		(property "Manufacturer_Part_Number" "FNGEPO002"
+			(at 392.43 941.63 0)
+			(effects
+				(font
+					(size 1.27 1.27)
+				)
+				(justify left top)
+				(hide yes)
+			)
+		)
+		(property "Mouser Part Number" "729-FNGEPO002"
+			(at 392.43 1041.63 0)
+			(effects
+				(font
+					(size 1.27 1.27)
+				)
+				(justify left top)
+				(hide yes)
+			)
+		)
+		(property "Mouser Price/Stock" "https://www.mouser.co.uk/ProductDetail/Diodes-Incorporated/FNGEPO002?qs=sggESLfvpWaEKfTCt%2F4zIA%3D%3D"
+			(at 392.43 1141.63 0)
+			(effects
+				(font
+					(size 1.27 1.27)
+				)
+				(justify left top)
+				(hide yes)
+			)
+		)
+		(property "Arrow Part Number" "FNGEPO002"
+			(at 392.43 1241.63 0)
+			(effects
+				(font
+					(size 1.27 1.27)
+				)
+				(justify left top)
+				(hide yes)
+			)
+		)
+		(property "Arrow Price/Stock" "https://www.arrow.com/en/products/fngepo002/diodes-incorporated"
+			(at 392.43 1341.63 0)
+			(effects
+				(font
+					(size 1.27 1.27)
+				)
+				(justify left top)
+				(hide yes)
+			)
+		)
+		(pin "1"
+		)
+		(pin "2"
+		)
+		(pin "3"
+		)
+		(pin "4"
+		)
+		(instances
+			(project ""
+				(path "/0ef51407-3c01-447a-a681-0fc3deaf4e2b"
+					(reference "Y1")
+					(unit 1)
+				)
