File: hardware/final-pcb/final-pcb/final-pcb.kicad_sch (KiCad schematic)
At the start: 0 parts

Commit message: Add syms, footprints, 3dmodels for ADS and LTC boards
Other:
- company: (none) -> San Diego State University
- title: (none) -> HANDS-EMG
Changed lines of the file:
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@@
 	(generator_version "8.0")
 	(paper "A4")
+	(title_block
+		(title "HANDS-EMG")
+		(date "2025-03-01")
+		(company "San Diego State University")
+		(comment 1 "Computer Engineer: Noah Marosok, Blake Pearson")
+		(comment 2 "Electrical Engineer: Kelly Hubbard, Jayden Sumbillo, Kirk Young")
+	)
 	(sheet
 		(at 88.9 25.4)
