File: hardware/final-pcb/final-pcb/final_handsEMG.kicad_sch (KiCad schematic)
At the start: 192 parts, among them J1 Conn_02x13_Odd_Even, U1 ADS1299CPAG, U2 STM32L496ZGT6, U3 FT231XQ-R, U6 TPS60403DBVT, U8 TPS72325DBVT, U9 TPS73225DBVT

Commit message: 90% of components are placed (4.5.25)
NEED TESTPOINTS and configure the jumper parts for the PMIC without using jumpers
Parts:
- L1, L2, L4, L5: footprint (none) -> MLZ2012A3R3W:INDC2012X87N
- U2: footprint STM32L496ZGT6:QFP50P2200X2200X160-144N -> STM32L496ZGT6:LQFP144-20x20mm_STM
- U6: footprint SOT95P280X145-5N -> TPS60403DBVT:SOT95P280X145-5N; Arrow Part Number TPS60403DBVT -> (none); Arrow Price/Stock https://www.arrow.com/en/products/tps60403dbvt/texas-instru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 -> (none); Height 1.45 -> (none); Manufacturer_Name Texas Instruments -> (none); Manufacturer_Part_Number TPS60403DBVT -> (none); Mouser Part Number 595-TPS60403DBVT -> (none); Mouser Price/Stock https://www.mouser.co.uk/ProductDetail/Texas-Instruments/TP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 -> (none)
- U9: footprint SOT95P280X145-5N -> TPS73225DBVT:SOT95P280X145-5N; Arrow Part Number TPS73225DBVT -> (none); Arrow Price/Stock https://www.arrow.com/en/products/tps73225dbvt/texas-instru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 -> (none); Height 1.45 -> (none); Manufacturer_Name Texas Instruments -> (none); Manufacturer_Part_Number TPS73225DBVT -> (none); Mouser Part Number 595-TPS73225DBVT -> (none); Mouser Price/Stock https://www.mouser.co.uk/ProductDetail/Texas-Instruments/TP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 -> (none)
- dL2: renamed from L3; footprint (none) -> MPZ1005S300C:IND_1005_TDK
- pC1, pC11, pC4, pC5, pC8, pC9: footprint (none) -> 03PowerFOOTPRINTS:C1005X5R0J105M
- pC10: footprint (none) -> 03PowerFOOTPRINTS:C1608X5R0J225M
- pC12: value 100uF -> 10uF; footprint (none) -> 03PowerFOOTPRINTS:C1608X5R0J106M
- pC13: footprint (none) -> 03PowerFOOTPRINTS:GRM31CR60J107ME39L
- pC14: footprint (none) -> 03PowerFOOTPRINTS:LMK316BJ476ML-T
- pC15, pC20, pC22, pC24: footprint (none) -> 03PowerFOOTPRINTS:04025A100KAT
- pC16, pC26, pC27, pC28, pC29: footprint (none) -> 03PowerFOOTPRINTS:C1005X5R1C104K
- pC17: footprint (none) -> 03PowerFOOTPRINTS:04025A331KAT
- pC18: footprint (none) -> 03PowerFOOTPRINTS:04025A330KAT
- pC19, pC6, pC7: footprint (none) -> 03PowerFOOTPRINTS:JMK212BJ226MG-T
- pC2: footprint (none) -> 03PowerFOOTPRINTS:GRM21BR61A106KE19
- pC21, pC23: footprint (none) -> 03PowerFOOTPRINTS:C1608X5R0J106M
- pC3: footprint (none) -> 03PowerFOOTPRINTS:GRM21BR61A106KE19L
- pD2: footprint (none) -> SMD-LED-CLEAR-GREEN_0603_:LED-0603
- pD3: footprint (none) -> LED-SMD-RED-DIFFUSED_0603_:LED-0603
- pJP2, pJP3, pJP4, pJP5, pJP6, pJP7, pJP8: footprint (none) -> 03PowerFOOTPRINTS:SAMTEC-TMM-103-02-X-S
- pL1: footprint (none) -> 03PowerFOOTPRINTS:LPS4018-332MLC
- pL2, pL3: footprint (none) -> 03PowerFOOTPRINTS:LPS4018-222MLC
- pL4, pL5: footprint (none) -> 03PowerFOOTPRINTS:IND_3010_TDK
- pQ1: footprint (none) -> 03PowerFOOTPRINTS:SI2333DS
- pR10, pR12, pR4: footprint (none) -> 03PowerFOOTPRINTS:CRCW04020000Z0EDC
- pR13, pR18, pR23, pR26: footprint (none) -> 03PowerFOOTPRINTS:CRCW040220R0FKED
- pR14: footprint (none) -> 03PowerFOOTPRINTS:CRCW040288K7FKED
- pR15: footprint (none) -> 03PowerFOOTPRINTS:CRCW040216K9FKED
- pR16: footprint (none) -> 03PowerFOOTPRINTS:CRCW04023K01FKED
- pR17: footprint (none) -> 03PowerFOOTPRINTS:CRCW04022K00FKED
- pR19: footprint (none) -> 03PowerFOOTPRINTS:CRCW040215K0FKED
- pR2, pR29, pR30, pR31: footprint (none) -> 03PowerFOOTPRINTS:CRCW04021R00JNED
- pR20: footprint (none) -> 03PowerFOOTPRINTS:CRCW0402324KFKED
- pR21: footprint (none) -> 03PowerFOOTPRINTS:CRCW0402121KFKED
- pR22: footprint (none) -> 03PowerFOOTPRINTS:CRCW0402105KFKED
- pR24: footprint (none) -> 03PowerFOOTPRINTS:CRCW0402806KFKED
- pR25: footprint (none) -> 03PowerFOOTPRINTS:CRCW0402649KFKED
- pR27: footprint (none) -> 03PowerFOOTPRINTS:CRCW0402232KFKED
- pR28: footprint (none) -> 03PowerFOOTPRINTS:CRCW0402464KFKED
- pR3, pR9: footprint (none) -> 03PowerFOOTPRINTS:CRCW0402100KFKED
- pR32, pR33, pR34, pR35, pR5, pR7: footprint (none) -> 03PowerFOOTPRINTS:CRCW04021K00JNED
- pR6, pR8: footprint (none) -> 03PowerFOOTPRINTS:CRCW04022K20FKED
- pU1: footprint (none) -> 03PowerFOOTPRINTS:LTC3586EUFE
- sC42: footprint (none) -> TAJA475K016R:CAPMP3216X166
- sJ2: footprint (none) -> S2B-PH-K-S:CONN_S2B-PH-K-S_JST
Connections:
- net -5VCC is gone; now on net -5V: C49.1, C50.1, C63.1, L2.2, U6.1 (OUT), U8.2 (IN), U8.3 (EN)
- net 5VCC is gone; now on net +5V: C46.1, C47.1, C58.1, L1.2, U6.2 (IN), U9.1 (IN), U9.3 (EN)
- net AVBUS: now also sR54.2
- net USB_VBUS: no longer sR54.2
