File: hardware/final-pcb/final-pcb/final_handsEMG.kicad_pcb (KiCad board)
At the start: 4 copper layers, 85.9 x 94.4 mm, 195 parts, among them J1 Conn_02x13_Odd_Even, U1 ADS1299CPAG, U2 STM32L496ZGT6, U3 LTC3586EUFE-3-PBF, U4 FT231XQ-R, U6 TPS60403DBVT, U8 TPS72325DBVT, U9 TPS73225DBVT

Commit message: lol forgot buttons (4.16.25)
Parts:
- added RESET: TS02-66-60-BK-160-LCR-D, FSM6JSMATR:SW_5-1437565-0, F.Cu at (84.3, 64.3)
- added USER: TS02-66-60-BK-160-LCR-D, FSM6JSMATR:SW_5-1437565-0, F.Cu at (133.0, 121.1)
- added sC40: [N/A], CC0402KRX7R7BB104:YAG_CC0402_YAG, F.Cu at (123.4, 111.4)
- added sC41: 100nF, CC0402KRX7R7BB104:YAG_CC0402_YAG, F.Cu at (82.5, 72.9)
- added sR42: 220K, RC0603FR-07220KL:RESC1607X60N, F.Cu at (123.4, 107.1)
- added sR43: 330, RC0603FR-07330RL:RESC1607X60N, F.Cu at (123.4, 109.7)
- added sR44: 100, RC0603FR-07100RL:RESC1607X60N, F.Cu at (123.4, 113.1)
- renumbered BAT to sJ2
Routing:
- net DGND: track 176.0 -> 213.2 mm
- net PC13: track 0.00 -> 33.6 mm, vias 0 -> 2
- net NRST: track 39.2 -> 63.9 mm
- net Net-(USER1-Pad1): track 0.00 -> 24.1 mm
- net AVOUT3: track 144.7 -> 154.4 mm, vias 26 -> 29
- net Net-(sC40-Pad2): track 0.00 -> 1.82 mm
