File: hardware/final-pcb/final-pcb/final_handsEMG.kicad_pcb (KiCad board)
At the start: 4 copper layers, 85.9 x 94.4 mm, 202 parts, among them J1 Conn_02x13_Odd_Even, U1 ADS1299CPAG, U2 STM32L496ZGT6, U3 LTC3586EUFE-3-PBF, U4 FT231XQ-R, U6 TPS60403DBVT, U8 TPS72325DBVT, U9 TPS73225DBVT

Commit message: implemented blakes revisions (4.21.25)
Parts:
- removed RESET, USER: TS02-66-60-BK-160-LCR-D, FSM6JSMATR:SW_5-1437565-0
- added pR80: 10K, 03PowerFOOTPRINTS:CRCW04021K00JNED, F.Cu at (122.5, 63.4)
- added pR81: 10K, 03PowerFOOTPRINTS:CRCW04021K00JNED, F.Cu at (122.5, 65.1)
- added pR82: 10K, 03PowerFOOTPRINTS:CRCW04021K00JNED, F.Cu at (122.5, 66.8)
- added pR83: 10K, 03PowerFOOTPRINTS:CRCW04021K00JNED, F.Cu at (122.5, 68.4)
- added sB1: USER, PTS645SH50SMTR92 LFS:PTS645S_SMTR92_CNK, F.Cu at (133.3, 121.6)
- added sB2: RESET, PTS645SH50SMTR92 LFS:PTS645S_SMTR92_CNK, F.Cu at (84.5, 64.1)
- added sR55: 10K (DNP), RC0603FR-0710KL:RESC1607X60N, F.Cu at (122.0, 121.0)
- U3: footprint 03PowerFOOTPRINTS:LTC3586EUFE -> LTC3586 Fixed:QFN-38_UFE_LIT
- sR54: value 10K -> 10K (DNP)
- renumbered SWD to SWD1
Connections:
- U2 pad 111: MODE -> PC10
- U2 pad 112: ILIM1 -> PC11
- U2 pad 113: ILIM0 -> PC12
- U2 pad 114: *FAULT -> PD0
- sCN14 pad 4: PA10 -> USB_ID
- sD6 pad 1: PA10 -> USB_ID
Routing:
- net PVIN3: track 81.3 -> 131.2 mm, vias 5 -> 9
- net PD0: track 0.00 -> 45.9 mm, vias 0 -> 2
- net PC12: track 0.00 -> 43.2 mm, vias 0 -> 2
- net PC11: track 0.00 -> 40.7 mm, vias 0 -> 2
- net PC10: track 0.00 -> 37.2 mm, vias 0 -> 2
- net USB_ID: track 0.00 -> 24.0 mm
- net *FAULT: track 84.4 -> 70.4 mm
- net ILIM1: track 53.6 -> 41.9 mm
- net ILIM0: track 57.0 -> 46.0 mm
- net MODE: track 58.0 -> 49.8 mm
- net AVDD: track 142.0 -> 146.2 mm, vias 11 -> 12
- net Net-(sB1-Pad1): track 24.1 -> 27.2 mm
- net BIAS: track 11.0 -> 13.6 mm
- net PA10: track 52.9 -> 51.1 mm
- net EN1: track 67.9 -> 69.5 mm
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
Commit message: labeled battery (4.21.25)
Parts:
- renumbered sJ2 to BAT
Other:
- board text added: "- +"
Changed lines of the file:
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@@
 		(at 157.7601 65.4851 90)
 		(tags "S2B-PH-K-SLFSN ")
-		(property "Reference" "sJ2"
+		(property "Reference" "BAT"
 			(at -3.3049 3.9019 0)
 			(unlocked yes)
@@
 			)
 			(justify left bottom)
+		)
+	)
+	(gr_text "-\n+"
+		(at 154.71 65.75 0)
+		(layer "F.SilkS")
+		(effects
+			(font
+				(size 1 1)
+				(thickness 0.1524)
+			)
+			(justify left bottom)
